Commit message: updating robody urdf

File: urdf/robody.xacro (robot description, xacro)
@@ -50,4 +50,5 @@
     </plugin>
   </gazebo>
+  <!-- ROBODYS BODY -->
   <link name="link_chassis">
     <!-- pose and inertial -->
@@ -58,8 +59,21 @@
       <inertia ixx="0.0395416666667" ixy="0" ixz="0" iyy="0.106208333333" iyz="0" izz="0.106208333333"/>
     </inertial>
+    <!-- base -->
+    <collision name="collision_base">
+      <geometry>
+        <box size="0.5 0.3 0.1" xyz="0 0 -0.3"/>
+      </geometry>
+    </collision>
+    <visual>
+      <origin rpy="0 0 0" xyz="0 0 -0.4"/>
+      <geometry>
+        <box size="0.5 0.3 0.1"/>
+      </geometry>
+      <material name="blue"/>
+    </visual>
     <!-- body -->
-    <collision name="collision_chassis">
-      <geometry>
-        <box size="0.5 0.3 3"/>
+    <collision name="collision_body">
+      <geometry>
+        <box size="0.25 0.25 0.8"/>
       </geometry>
     </collision>
@@ -67,11 +81,11 @@
       <origin rpy="0 0 0" xyz="0 0 0"/>
       <geometry>
-        <box size="0.5 0.3 3"/>
+        <box size="0.25 0.25 0.8"/>
       </geometry>
       <material name="blue"/>
     </visual>
-    <!-- caster front -->
-    <collision name="caster_front_collision">
-      <origin rpy=" 0 0 0" xyz="0.35 0 -0.05"/>
+    <!-- caster front right -->
+    <collision name="caster_front_right_collision">
+      <origin rpy=" 0 0 0" xyz="0.35 0.15 -0.53"/>
       <geometry>
         <sphere radius="0.05"/>
@@ -82,17 +96,86 @@
             <mu>0</mu>
             <mu2>0</mu2>
-            <slip1>1.0</slip1>
-            <slip2>1.0</slip2>
+            <slip1>2.0</slip1>
+            <slip2>2.0</slip2>
           </ode>
         </friction>
       </surface>
     </collision>
-    <visual name="caster_front_visual">
-      <origin rpy=" 0 0 0" xyz="0.2 0 -0.05"/>
-      <geometry>
-        <sphere radius="0.05"/>
-      </geometry>
-    </visual>
-  </link>
+    <visual name="caster_front_right_visual">
+      <origin rpy=" 0 0 0" xyz="0.2 0.15 -0.53"/>
+      <geometry>
+        <sphere radius="0.05"/>
+      </geometry>
+    </visual>
+    <!-- caster front left -->
+    <collision name="caster_front_left_collision">
+      <origin rpy=" 0 0 0" xyz="0.35 -0.15 -0.53"/>
+      <geometry>
+        <sphere radius="0.05"/>
+      </geometry>
+      <surface>
+        <friction>
+          <ode>
+            <mu>0</mu>
+            <mu2>0</mu2>
+            <slip1>2.0</slip1>
+            <slip2>2.0</slip2>
+          </ode>
+        </friction>
+      </surface>
+    </collision>
+    <visual name="caster_front_left_visual">
+      <origin rpy=" 0 0 0" xyz="0.2 -0.15 -0.53"/>
+      <geometry>
+        <sphere radius="0.05"/>
+      </geometry>
+    </visual>
+  <!-- caster back right -->
+    <collision name="caster_back_right_collision">
+        <origin rpy=" 0 0 0" xyz="-0.35 0.15 -0.53"/>
+        <geometry>
+        <sphere radius="0.05"/>
+        </geometry>
+        <surface>
+        <friction>
+            <ode>
+            <mu>0</mu>
+            <mu2>0</mu2>
+            <slip1>2.0</slip1>
+            <slip2>2.0</slip2>
+            </ode>
+        </friction>
+        </surface>
+    </collision>
+    <visual name="caster_back_right_visual">
+        <origin rpy=" 0 0 0" xyz="-0.2 0.15 -0.53"/>
+        <geometry>
+        <sphere radius="0.05"/>
+        </geometry>
+    </visual>
+    <!-- caster back left -->
+    <collision name="caster_back_left_collision">
+      <origin rpy=" 0 0 0" xyz="-0.35 -0.15 -0.53"/>
+      <geometry>
+        <sphere radius="0.05"/>
+      </geometry>
+      <surface>
+        <friction>
+          <ode>
+            <mu>0</mu>
+            <mu2>0</mu2>
+            <slip1>2.0</slip1>
+            <slip2>2.0</slip2>
+          </ode>
+        </friction>
+      </surface>
+    </collision>
+    <visual name="caster_back_left_visual">
+      <origin rpy=" 0 0 0" xyz="-0.2 -0.15 -0.53"/>
+      <geometry>
+        <sphere radius="0.05"/>
+      </geometry>
+    </visual>
+</link>
   <link name="link_right_wheel">
     <inertial>
@@ -115,5 +198,5 @@
   </link>
   <joint name="joint_right_wheel" type="continuous">
-    <origin rpy="0 0 0" xyz="-0.05 0.15 0"/>
+    <origin rpy="0 0 0" xyz="-0.05 0.15 -0.5"/>
     <child link="link_right_wheel"/>
     <parent link="link_chassis"/>
@@ -142,5 +225,5 @@
   </link>
   <joint name="joint_left_wheel" type="continuous">
-    <origin rpy="0 0 0" xyz="-0.05 -0.15 0"/>
+    <origin rpy="0 0 0" xyz="-0.05 -0.15 -0.5"/>
     <child link="link_left_wheel"/>
     <parent link="link_chassis"/>
